Commit message: Upload 25.12.23

File: Explanation-of-URDF-Files-and-Launch-ROS-Files/robot_ws/src/robot_model_pkg/urdf/robot.urdf (robot description, URDF)
Before this commit: robot simple_robot, 1 links, 0 joints
Links:
- added link first_link; visual cylinder length=0.5 radius=0.04
- added link second_link; visual box size=0.1 1 0.1
Joints:
- added joint joint_1: type revolute, parent base_link, child first_link, origin xyz=0 0 0.025, axis 0 0 1, limit lower=-1.2 upper=1.2 effort=300 velocity=2.0
- added joint joint_2: type prismatic, parent first_link, child second_link, origin xyz=0 0 0.5, axis 0 1 0, limit lower=-5 upper=5 effort=300 velocity=2.0
