Commit message: Upload 14.2.24

File: Modelling-Simulation-and-Control-of-2-Wheeled-Robot-in-ROS-and-Gazebo/robot_two_wheeled/src/robot_model_pkg/urdf/robot.xacro (robot description, xacro)
@@ -335,10 +335,10 @@
     <!-- Second four support sticks of our robot -->
     <!-- ####################################### -->
-<!-- belirlediğimiz origin değeri öbjenin başlangıcı değil objenin merkezi imiş, diğer tüm değerli kontrol etmem lazımi bundan sonrakileri buna dikkat ederecek yapmalıyım önemli not. henüz düzenlenmediler -->
+<!-- belirlediğimiz origin değeri öbjenin başlangıcı imiş, diğer tüm değerli kontrol etmem lazımi bundan sonrakileri buna dikkat ederecek yapmalıyım önemli not. henüz düzenlenmediler -->
     <!-- Left front -->
     <joint name="upper_body_support_lf_2" type="fixed">
         <parent link="upper_body_1_link"/>
         <child link="upper_body_support_lf_2_link"/>
-        <origin xyz="-0.0155 -0.033 0.04" rpy="0.0 0.0 0.0"/>
+        <origin xyz="-0.0155 -0.033 0.08" rpy="0.0 0.0 0.0"/>
         <axis xyz="0.0 0.0 0.0"/>
         <limit lower="0.0" upper="0.0" effort="0.0" velocity="0.0"/>
@@ -346,11 +346,11 @@
     <link name="upper_body_support_lf_2_link">
         <visual>
-            <origin xyz="-0.0155 -0.033 0.04" rpy="0.0 0.0 0.0"/>
-            <geometry>
-                <box size="0.01 0.01 0.03"/>
-            </geometry>
-        </visual>
-        <collision>
-            <origin xyz="-0.0155 -0.033 0.04" rpy="0.0 0.0 0.0"/>
+            <origin xyz="-0.0155 -0.033 0.08" rpy="0.0 0.0 0.0"/>
+            <geometry>
+                <box size="0.01 0.01 0.03"/>
+            </geometry>
+        </visual>
+        <collision>
+            <origin xyz="-0.0155 -0.033 0.08" rpy="0.0 0.0 0.0"/>
             <geometry>
                 <box size="0.01 0.01 0.03"/>
@@ -364,5 +364,5 @@
         <parent link="upper_body_1_link"/>
         <child link="upper_body_support_lb_2_link"/>
-        <origin xyz="-0.0565 -0.033 0.04" rpy="0.0 0.0 0.0"/>
+        <origin xyz="-0.0565 -0.033 0.08" rpy="0.0 0.0 0.0"/>
         <axis xyz="0.0 0.0 0.0"/>
         <limit lower="0.0" upper="0.0" effort="0.0" velocity="0.0"/>
@@ -370,11 +370,11 @@
     <link name="upper_body_support_lb_2_link">
         <visual>
-            <origin xyz="-0.0565 -0.033 0.04" rpy="0.0 0.0 0.0"/>
-            <geometry>
-                <box size="0.01 0.01 0.03"/>
-            </geometry>
-        </visual>
-        <collision>
-            <origin xyz="-0.0565 -0.033 0.04" rpy="0.0 0.0 0.0"/>
+            <origin xyz="-0.0565 -0.033 0.08" rpy="0.0 0.0 0.0"/>
+            <geometry>
+                <box size="0.01 0.01 0.03"/>
+            </geometry>
+        </visual>
+        <collision>
+            <origin xyz="-0.0565 -0.033 0.08" rpy="0.0 0.0 0.0"/>
             <geometry>
                 <box size="0.01 0.01 0.03"/>
@@ -388,5 +388,5 @@
         <parent link="upper_body_1_link"/>
         <child link="upper_body_support_rf_2_link"/>
-        <origin xyz="-0.0155 0.033 0.04" rpy="0.0 0.0 0.0"/>
+        <origin xyz="-0.0155 0.033 0.08" rpy="0.0 0.0 0.0"/>
         <axis xyz="0.0 0.0 0.0"/>
         <limit lower="0.0" upper="0.0" effort="0.0" velocity="0.0"/>
@@ -394,11 +394,11 @@
     <link name="upper_body_support_rf_2_link">
         <visual>
-            <origin xyz="-0.0155 0.033 0.04" rpy="0.0 0.0 0.0"/>
-            <geometry>
-                <box size="0.01 0.01 0.03"/>
-            </geometry>
-        </visual>
-        <collision>
-            <origin xyz="-0.0155 0.033 0.04" rpy="0.0 0.0 0.0"/>
+            <origin xyz="-0.0155 0.033 0.08" rpy="0.0 0.0 0.0"/>
+            <geometry>
+                <box size="0.01 0.01 0.03"/>
+            </geometry>
+        </visual>
+        <collision>
+            <origin xyz="-0.0155 0.033 0.08" rpy="0.0 0.0 0.0"/>
             <geometry>
                 <box size="0.01 0.01 0.03"/>
@@ -412,5 +412,5 @@
         <parent link="upper_body_1_link"/>
         <child link="upper_body_support_rb_2_link"/>
-        <origin xyz="-0.0565 0.033 0.04" rpy="0.0 0.0 0.0"/>
+        <origin xyz="-0.0565 0.033 0.08" rpy="0.0 0.0 0.0"/>
         <axis xyz="0.0 0.0 0.0"/>
         <limit lower="0.0" upper="0.0" effort="0.0" velocity="0.0"/>
@@ -418,17 +418,43 @@
     <link name="upper_body_support_rb_2_link">
         <visual>
-            <origin xyz="-0.0565 0.033 0.04" rpy="0.0 0.0 0.0"/>
-            <geometry>
-                <box size="0.01 0.01 0.03"/>
-            </geometry>
-        </visual>
-        <collision>
-            <origin xyz="-0.0565 0.033 0.04" rpy="0.0 0.0 0.0"/>
-            <geometry>
-                <box size="0.01 0.01 0.03"/>
-            </geometry>
-        </collision>
-        <!-- Macro we defined before -->
-        <xacro:inertia_upper_body_support>
+            <origin xyz="-0.0565 0.033 0.08" rpy="0.0 0.0 0.0"/>
+            <geometry>
+                <box size="0.01 0.01 0.03"/>
+            </geometry>
+        </visual>
+        <collision>
+            <origin xyz="-0.0565 0.033 0.08" rpy="0.0 0.0 0.0"/>
+            <geometry>
+                <box size="0.01 0.01 0.03"/>
+            </geometry>
+        </collision>
+        <!-- Macro we defined before -->
+        <xacro:inertia_upper_body_support>
+    </link>
+    <!-- ############################## -->
+    <!-- Second upper body of our robot -->
+    <!-- ############################## -->
+    <joint name="upper_body_2_joint" type="fixed">
+        <parent link="upper_body_support_lf_2_link"/>
+        <child link="upper_body_2_link"/>
+        <origin xyz="-0.036 0.0 0.15" rpy="0.0 0.0 0.0"/>
+        <axis xyz="0.0 0.0 0.0"/>
+        <limit lower="0.0" upper="0.0" effort="0.0" velocity="0.0"/>
+    </joint>
+    <link name="upper_body_2_link">
+        <visual>
+            <origin xyz="-0.036 0.0 0.15" rpy="0.0 0.0 0.0"/>
+            <geometry>
+                <box size="0.055 0.08 0.01"/>
+            </geometry>
+        </visual>
+        <collision>
+            <origin xyz="-0.036 0.0 0.15" rpy="0.0 0.0 0.0"/>
+            <geometry>
+                <box size="0.055 0.08 0.01"/>
+            </geometry>
+        </collision>
+        <!-- Macro we defined before -->
+        <xacro:inertia_upper_body>
     </link>
 </robot>

Commit message: Upload 14.2.24

File: Modelling-Simulation-and-Control-of-2-Wheeled-Robot-in-ROS-and-Gazebo/robot_two_wheeled/src/robot_model_pkg/urdf/robot.xacro (robot description, xacro)
@@ -26,5 +26,5 @@
     <xacro:property name="support_wheel_body_link_z_dim" value="0.010"/>
     <!-- Support Wheel Dimension -->
-    <xacro:property name="support_wheel_link_radius" value="0.005"/>
+    <xacro:property name="support_wheel_link_radius" value="0.5"/> <!-- 0.005 idi -->
     <xacro:property name="support_wheel_link_length" value="0.1"/>
     <xacro:property name="support_wheel_link_z_location" value="0.010"/>
@@ -35,10 +35,10 @@
     <xacro:property name="pi_const" value="3.14159265"/>
     <!-- Robot body and wheel mass -->
-    <xacro:property name="body_mass" value="$ {body_density*body_link_x_dim*body_link_y_dim*body_link_z_dim}"/>
+    <xacro:property name="body_mass" value="${body_density*body_link_x_dim*body_link_y_dim*body_link_z_dim}"/>
     <xacro:property name="wheel_mass" value="${wheel_density*pi_const*wheel_link_radius*wheel_link_radius*wheel_link_length}"/>
-    <xacro:property name="upper_body_mass" value="body_density*upper_body_link_x_dim*upper_body_link_y_dim*upper_body_link_z_dim"/>
-    <xacro:property name="upper_body_support_mass" value="body_mass*upper_body_support_link_x_dim*upper_body_support_link_y_dim*upper_body_support_link_z_dim"/>
-    <xacro:property name="support_wheel_body_mass" value="body_mass*support_wheel_body_link_x_dim*support_wheel_body_link_y_dim*support_wheel_body_link_z_dim"/>
-    <xacro:property name="support_wheel_mass" value="wheel_density*pi_const*(support_wheel_link_radius/2)*(support_wheel_link_radius/2)*support_wheel_link_length"/>
+    <xacro:property name="upper_body_mass" value="${body_density*upper_body_link_x_dim*upper_body_link_y_dim*upper_body_link_z_dim}"/>
+    <xacro:property name="upper_body_support_mass" value="${body_mass*upper_body_support_link_x_dim*upper_body_support_link_y_dim*upper_body_support_link_z_dim}"/>
+    <xacro:property name="support_wheel_body_mass" value="${body_mass*support_wheel_body_link_x_dim*support_wheel_body_link_y_dim*support_wheel_body_link_z_dim}"/>
+    <xacro:property name="support_wheel_mass" value="${wheel_density*pi_const*(support_wheel_link_radius/2.0)*(support_wheel_link_radius/2.0)*support_wheel_link_length}"/>
     <!-- Moments of inertia of the wheel -->
     <xacro:property name="Iz_wheel" value="${0.5*wheel_mass*wheel_link_radius*wheel_link_radius}"/>
@@ -57,5 +57,5 @@
             <origin xyz="0 0 0" rpy="0 0 0"/>
             <mass value="${upper_body_support_mass}"/>
-            <inertia ixx="${(1/12)*upper_body_support_mass*(upper_body_support_link_y_dim*upper_body_support_link_y_dim+upper_body_support_link_z_dim*upper_body_support_link_z_dim)}" ixy="0" ixz="0" iyy="${(1/12)*upper_body_support_mass*(upper_body_support_link_x_dim*upper_body_support_link_x_dim+upper_body_support_link_z_dim*upper_body_support_link_z_dim)}" iyz="0" izz="${(1/12)*upper_body_support_mass*(upper_body_support_link_x_dim*upper_body_support_link_x_dim+upper_body_support_link_y_dim*upper_body_support_link_y_dim)}"/>
+            <inertia ixx="${(1.0/12.0)*upper_body_support_mass*(upper_body_support_link_y_dim*upper_body_support_link_y_dim+upper_body_support_link_z_dim*upper_body_support_link_z_dim)}" ixy="0" ixz="0" iyy="${(1.0/12.0)*upper_body_support_mass*(upper_body_support_link_x_dim*upper_body_support_link_x_dim+upper_body_support_link_z_dim*upper_body_support_link_z_dim)}" iyz="0" izz="${(1.0/12.0)*upper_body_support_mass*(upper_body_support_link_x_dim*upper_body_support_link_x_dim+upper_body_support_link_y_dim*upper_body_support_link_y_dim)}"/>
         </inertial>
     </xacro:macro>
@@ -64,5 +64,5 @@
             <origin xyz="0 0 0" rpy="0 0 0"/>
             <mass value="${upper_body_mass}"/>
-            <inertia ixx="${(1/12)*upper_body_mass*(upper_body_link_y_dim*upper_body_link_y_dim+upper_body_link_z_dim*upper_body_link_z_dim)}" ixy="0" ixz="0" iyy="${(1/12)*upper_body_mass*(upper_body_link_x_dim*upper_body_link_x_dim+upper_body_link_z_dim*upper_body_link_z_dim)}" iyz="0" izz="${(1/12)*upper_body_mass*(upper_body_link_x_dim*upper_body_link_x_dim+upper_body_link_y_dim*upper_body_link_y_dim)}"/>
+            <inertia ixx="${(1.0/12.0)*upper_body_mass*(upper_body_link_y_dim*upper_body_link_y_dim+upper_body_link_z_dim*upper_body_link_z_dim)}" ixy="0" ixz="0" iyy="${(1.0/12.0)*upper_body_mass*(upper_body_link_x_dim*upper_body_link_x_dim+upper_body_link_z_dim*upper_body_link_z_dim)}" iyz="0" izz="${(1.0/12.0)*upper_body_mass*(upper_body_link_x_dim*upper_body_link_x_dim+upper_body_link_y_dim*upper_body_link_y_dim)}"/>
         </inertial>
     </xacro:macro>
@@ -100,5 +100,5 @@
             <origin xyz="0.0 0.0 0.0" rpy="0.0 0.0 0.0"/>
             <mass value="${body_mass}"/>
-            <inertia ixx="${(1/12)*body_mass*(body_link_y_dim*body_link_y_dim+body_link_z_dim*body_link_z_dim)}" ixy="0" ixz="0" iyy="${(1/12)*body_mass*(body_link_x_dim*body_link_x_dim+body_link_z_dim*body_link_z_dim)}" iyz="0" izz="${(1/12)*body_mass*(body_link_y_dim*body_link_y_dim+body_link_x_dim*body_link_x_dim)}"/>
+            <inertia ixx="${(1.0/12.0)*body_mass*(body_link_y_dim*body_link_y_dim+body_link_z_dim*body_link_z_dim)}" ixy="0" ixz="0" iyy="${(1.0/12.0)*body_mass*(body_link_x_dim*body_link_x_dim+body_link_z_dim*body_link_z_dim)}" iyz="0" izz="${(1.0/12.0)*body_mass*(body_link_y_dim*body_link_y_dim+body_link_x_dim*body_link_x_dim)}"/>
         </inertial>
     </link>
@@ -107,5 +107,5 @@
     <!-- ################### -->
     <!-- Right Wheel -->
-    <joint name="wheel_right_joint" type="continious">
+    <joint name="wheel_right_joint" type="continuous">
         <parent link="body_link"/>
         <child link="wheel_right_link"/>
@@ -129,8 +129,8 @@
         </collision>
         <!-- Macro we defined before -->
-        <xacro:inertia_wheel>
+        <xacro:inertia_wheel/>
     </link>
     <!-- Left Wheel -->
-    <joint name="wheel_left_joint" type="continious">
+    <joint name="wheel_left_joint" type="continuous">
         <parent link="body_link"/>
         <child link="wheel_left_link"/>
@@ -154,5 +154,5 @@
         </collision>
         <!-- Macro we defined before -->
-        <xacro:inertia_wheel>
+        <xacro:inertia_wheel/>
     </link>
     <!-- Support Wheel Body -->
@@ -180,5 +180,5 @@
     </link>
     <!-- Support Wheel -->
-    <joint name="support_wheel_joint" type="continious">
+    <joint name="support_wheel_joint" type="continuous">
         <parent link="support_wheel_body_link"/>
         <child link="support_wheel_link"/>
@@ -192,5 +192,5 @@
             <origin xyz="-0.047 0.0 0.015" rpy="1.2345 0.56789 0.392699"/>
             <geometry>
-                <sphere radius="0.005"/>
+                <sphere radius="support_wheel_link_radius"/>
             </geometry>
         </visual>
@@ -198,5 +198,5 @@
             <origin xyz="-0.047 0.0 0.015" rpy="1.2345 0.56789 0.392699"/>
             <geometry>
-                <sphere radius="0.005"/>
+                <sphere radius="support_wheel_link_radius"/>
             </geometry>
         </collision>
@@ -204,5 +204,5 @@
             <origin xyz="-0.047 0.0 0.015" rpy="1.2345 0.56789 0.392699"/>
             <mass value="${body_mass}"/>
-            <inertia ixx="${(2/5)*support_wheel_mass*0.005^2}" ixy="0" ixz="0" iyy="${(2/5)*support_wheel_mass*0.005^2}" iyz="0" izz="${(2/5)*support_wheel_mass*0.005^2}"/>
+            <inertia ixx="${(2.0/5.0)*support_wheel_mass*support_wheel_link_radius*support_wheel_link_radius}" ixy="0" ixz="0" iyy="${(2.0/5.0)*support_wheel_mass*0.005*0.005}" iyz="0" izz="${(2.0/5.0)*support_wheel_mass*0.005*0.005}"/>
         </inertial>
     </link>
@@ -211,5 +211,5 @@
     <!-- ###################################### -->
     <!-- Left front -->
-    <joint name="upper_body_support_lf" type="fixed">
+    <joint name="upper_body_support_lf_joint" type="fixed">
         <parent link="body_link"/>
         <child link="upper_body_support_lf_link"/>
@@ -232,8 +232,8 @@
         </collision>
         <!-- Macro we defined before -->
-        <xacro:inertia_upper_body_support>
+        <xacro:inertia_upper_body_support/>
     </link>
     <!-- Left back -->
-    <joint name="upper_body_support_lb" type="fixed">
+    <joint name="upper_body_support_lb_joint" type="fixed">
         <parent link="body_link"/>
         <child link="upper_body_support_lb_link"/>
@@ -256,8 +256,8 @@
         </collision>
         <!-- Macro we defined before -->
-        <xacro:inertia_upper_body_support>
+        <xacro:inertia_upper_body_support/>
     </link>
     <!-- Right front -->
-    <joint name="upper_body_support_rf" type="fixed">
+    <joint name="upper_body_support_rf_joint" type="fixed">
         <parent link="body_link"/>
         <child link="upper_body_support_rf_link"/>
@@ -280,8 +280,8 @@
         </collision>
         <!-- Macro we defined before -->
-        <xacro:inertia_upper_body_support>
+        <xacro:inertia_upper_body_support/>
     </link>
     <!-- Right back -->
-    <joint name="upper_body_support_rb" type="fixed">
+    <joint name="upper_body_support_rb_joint" type="fixed">
         <parent link="body_link"/>
         <child link="upper_body_support_rb_link"/>
@@ -304,5 +304,5 @@
         </collision>
         <!-- Macro we defined before -->
-        <xacro:inertia_upper_body_support>
+        <xacro:inertia_upper_body_support/>
     </link>
     <!-- ############################# -->
@@ -310,5 +310,5 @@
     <!-- ############################# -->
     <joint name="upper_body_1_joint" type="fixed">
-        <parent link="upper_body_support_lf"/>
+        <parent link="upper_body_support_lf_link"/>
         <child link="upper_body_1_link"/>
         <origin xyz="-0.036 0.0 0.075" rpy="0.0 0.0 0.0"/>
@@ -330,5 +330,5 @@
         </collision>
         <!-- Macro we defined before -->
-        <xacro:inertia_upper_body>
+        <xacro:inertia_upper_body/>
     </link>
     <!-- ####################################### -->
@@ -337,5 +337,5 @@
 <!-- belirlediğimiz origin değeri öbjenin başlangıcı imiş, diğer tüm değerli kontrol etmem lazımi bundan sonrakileri buna dikkat ederecek yapmalıyım önemli not. henüz düzenlenmediler -->
     <!-- Left front -->
-    <joint name="upper_body_support_lf_2" type="fixed">
+    <joint name="upper_body_support_lf_2_joint" type="fixed">
         <parent link="upper_body_1_link"/>
         <child link="upper_body_support_lf_2_link"/>
@@ -358,8 +358,8 @@
         </collision>
         <!-- Macro we defined before -->
-        <xacro:inertia_upper_body_support>
+        <xacro:inertia_upper_body_support/>
     </link>
     <!-- Left back -->
-    <joint name="upper_body_support_lb_2" type="fixed">
+    <joint name="upper_body_support_lb_2_joint" type="fixed">
         <parent link="upper_body_1_link"/>
         <child link="upper_body_support_lb_2_link"/>
@@ -382,8 +382,8 @@
         </collision>
         <!-- Macro we defined before -->
-        <xacro:inertia_upper_body_support>
+        <xacro:inertia_upper_body_support/>
     </link>
     <!-- Right front -->
-    <joint name="upper_body_support_rf_2" type="fixed">
+    <joint name="upper_body_support_rf_2_joint" type="fixed">
         <parent link="upper_body_1_link"/>
         <child link="upper_body_support_rf_2_link"/>
@@ -406,8 +406,8 @@
         </collision>
         <!-- Macro we defined before -->
-        <xacro:inertia_upper_body_support>
+        <xacro:inertia_upper_body_support/>
     </link>
     <!-- Right back -->
-    <joint name="upper_body_support_rb_2" type="fixed">
+    <joint name="upper_body_support_rb_2_joint" type="fixed">
         <parent link="upper_body_1_link"/>
         <child link="upper_body_support_rb_2_link"/>
@@ -430,5 +430,5 @@
         </collision>
         <!-- Macro we defined before -->
-        <xacro:inertia_upper_body_support>
+        <xacro:inertia_upper_body_support/>
     </link>
     <!-- ############################## -->
@@ -456,5 +456,5 @@
         </collision>
         <!-- Macro we defined before -->
-        <xacro:inertia_upper_body>
+        <xacro:inertia_upper_body/>
     </link>
 </robot>
